File: hardware/opentone/dac.kicad_sch (KiCad schematic)
At the start: 35 parts, among them U701 CS43131-CNZ, U702 TPS7A2018PDBVR, U703 SN74AVC4T245PWR, U704 PCA9306DCUR

Commit message: updated BOM
Parts:
- C701, C702: LCSC (none) -> C15849; Manufacturer (none) -> Samsung Electro-Mechanics; Part number (none) -> CL10A105KB8NNNC
- C703: LCSC (none) -> C19666; Manufacturer (none) -> Samsung Electro-Mechanics; Part number (none) -> CL10A475KO8NNNC
- C704, C705, C706, C717, C718, C719: LCSC (none) -> C14663; Manufacturer (none) -> YAGEO; Part number (none) -> CC0603KRX7R9BB104
- C707, C708, C711, C712, C713, C714, C715, C716: LCSC (none) -> C23630; Manufacturer (none) -> Samsung Electro-Mechanics; Part number (none) -> CL10A225KO8NNNC
- C709, C710: LCSC (none) -> C45783; Manufacturer (none) -> Samsung Electro-Mechanics; Part number (none) -> CL21A226MAQNNNE
- JP701, NT701: now left out of the parts list
