File: hardware/opentone/opentone.kicad_sch (KiCad schematic)
At the start: 3 parts, among them U1 STM32F446RCTx

Commit message: devboard audio and bluetooth schema
Parts:
- removed SCREEN1: ~, opentone:nhd-2.4-240320cf-ctxif, symbol screen-40pins-ili9488:screen-ili9488
- removed S_CONNECTOR1: ~, opentone:Hirose_FH12-40S-0.5SH_1x40-1MP_P0.50mm_Horizontal, symbol screen-40pins-ili9488:connector
Other:
- sheet BT Devboard renamed Bluetooth
- removed sheet bluetooth
- added sheet Screens (screens.kicad_sch)
- sheet Bluetooth: file bt_devboard.kicad_sch -> bluetooth.kicad_sch

Commit message: wiring main MCU
Parts:
- removed U1: STM32F446RCTx, Package_QFP:LQFP-64_10x10mm_P0.5mm, symbol MCU_ST_STM32F4:STM32F446RCTx
Other:
- added sheet MCU (mcu.kicad_sch)

Commit message: updated buttons and MCU
Other:
- removed sheet click-wheel-base-devboard
Changed lines of the file:
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@@
 	)
 	(sheet
-		(at 19.05 113.03)
-		(size 20.32 8.89)
+		(at 160.02 60.96)
+		(size 50.8 25.4)
 		(exclude_from_sim no)
 		(in_bom yes)
@@
 			(color 0 0 0 0.0000)
 		)
-		(property "Sheetname" "click-wheel-base-devboard"
-			(at 19.05 112.3184 0)
+		(property "Sheetname" "MCU"
+			(at 160.02 60.2484 0)
 			(effects
 				(font
@@
 			)
 		)
-		(property "Sheetfile" "click-wheel-base-devboard.kicad_sch"
-			(at 19.05 122.5046 0)
+		(property "Sheetfile" "mcu.kicad_sch"
+			(at 160.02 86.9446 0)
 			(effects
 				(font
@@
 				)
 			)
-		)
-	)
-	(sheet
-		(at 160.02 60.96)
-		(size 50.8 25.4)
-		(exclude_from_sim no)
-		(in_bom yes)
-		(on_board yes)
-		(dnp no)
-		(fields_autoplaced yes)
-		(stroke
-			(width 0.1524)
-			(type solid)
-		)
-		(fill
-			(color 0 0 0 0.0000)
-		)
-		(property "Sheetname" "MCU"
-			(at 160.02 60.2484 0)
-			(effects
-				(font
-					(size 1.27 1.27)
-				)
-				(justify left bottom)
-			)
-		)
-		(property "Sheetfile" "mcu.kicad_sch"
-			(at 160.02 86.9446 0)
-			(effects
-				(font
-					(size 1.27 1.27)
-				)
-				(justify left top)
-			)
-		)
-		(instances
-			(project "opentone"
-				(path "/0122bb8c-dbef-4db1-a6c6-9be780a38d9f"
-					(page "8")
-				)
-			)

Commit message: added sd card, haptic, updated old parts and set a datasheet and MPN to all parts
Other:
- added sheet Memory (memory.kicad_sch)
Changed lines of the file:
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@@
 (kicad_sch
-	(version 20250114)
+	(version 20260306)
 	(generator "eeschema")
-	(generator_version "9.0")
+	(generator_version "10.0")
 	(paper "A4")
+	(sheet
+		(at 160.02 96.52)
+		(size 50.8 25.4)
+		(exclude_from_sim no)
+		(in_bom yes)
+		(on_board yes)
+		(dnp no)
+		(fields_autoplaced yes)
+		(stroke
+			(width 0.1524)
+			(type solid)
+		)
+		(fill
+			(color 0 0 0 0)
+		)
+		(property "Sheetname" "Memory"
+			(at 160.02 95.8084 0)
+			(show_name no)
+			(do_not_autoplace no)
+			(effects
+				(font
+					(size 1.27 1.27)
+				)
+				(justify left bottom)
+			)
+		)
+		(property "Sheetfile" "memory.kicad_sch"
+			(at 160.02 122.5046 0)
+			(show_name no)
+			(do_not_autoplace no)
+			(effects
+				(font
+					(size 1.27 1.27)
+				)
+				(justify left top)
+			)
+		)
+		(instances
+			(project "opentone"
+				(path "/0122bb8c-dbef-4db1-a6c6-9be780a38d9f"
+					(page "8")
+				)
+			)
+		)
+	)
 	(sheet
 		(at 18.288 62.484)
@@
 		)
 		(fill
-			(color 0 0 0 0.0000)
+			(color 0 0 0 0)
 		)
 		(property "Sheetname" "Audio"
 			(at 18.288 61.7724 0)
+			(show_name no)
+			(do_not_autoplace no)
 			(effects
 				(font
@@
 		(property "Sheetfile" "audio.kicad_sch"
 			(at 18.288 100.4066 0)
+			(show_name no)
+			(do_not_autoplace no)
 			(effects
 				(font
@@
 		)
 		(fill
-			(color 0 0 0 0.0000)
+			(color 0 0 0 0)
 		)
 		(property "Sheetname" "Screens"
 			(at 84.328 105.9684 0)
+			(show_name no)
+			(do_not_autoplace no)
 			(effects
 				(font
@@
 		(property "Sheetfile" "screens.kicad_sch"
 			(at 84.328 127.5846 0)
+			(show_name no)
+			(do_not_autoplace no)
 			(effects
 				(font
@@
 		)
 		(fill
-			(color 0 0 0 0.0000)
+			(color 0 0 0 0)
 		)
 		(property "Sheetname" "Buttons"
 			(at 82.296 21.6404 0)
+			(show_name no)
+			(do_not_autoplace no)
 			(effects
 				(font
@@
 		(property "Sheetfile" "buttons.kicad_sch"
 			(at 82.296 57.9886 0)
+			(show_name no)
+			(do_not_autoplace no)
 			(effects
 				(font
@@
 		)
 		(fill
-			(color 0 0 0 0.0000)
+			(color 0 0 0 0)
 		)
 		(property "Sheetname" "MCU"
 			(at 160.02 60.2484 0)
+			(show_name no)
+			(do_not_autoplace no)
 			(effects
 				(font
@@
 		(property "Sheetfile" "mcu.kicad_sch"
 			(at 160.02 86.9446 0)
+			(show_name no)
+			(do_not_autoplace no)
 			(effects
 				(font
@@
 		)
 		(fill
-			(color 0 0 0 0.0000)
+			(color 0 0 0 0)
 		)
 		(property "Sheetname" "Power"
 			(at 18.034 18.0844 0)
+			(show_name no)
+			(do_not_autoplace no)
 			(effects
 				(font
@@
 		(property "Sheetfile" "power.kicad_sch"
 			(at 18.034 56.7186 0)
+			(show_name no)
+			(do_not_autoplace no)
 			(effects
 				(font
@@
 		)
 		(fill
-			(color 0 0 0 0.0000)
+			(color 0 0 0 0)
 		)
 		(property "Sheetname" "Bluetooth"
 			(at 83.058 63.2964 0)
+			(show_name no)
+			(do_not_autoplace no)
 			(effects
 				(font
@@
 		(property "Sheetfile" "bluetooth.kicad_sch"
 			(at 83.058 94.8186 0)
-			(effects
-				(font
+			(show_name no)
+			(do_not_autoplace no)
+			(effects
+				(font

Commit message: DAC
Other:
- added sheet DAC (dac.kicad_sch)
Changed lines of the file:
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@@
+	)
+	(sheet
+		(at 18.034 106.68)
+		(size 55.118 25.4)
+		(exclude_from_sim no)
+		(in_bom yes)
+		(on_board yes)
+		(dnp no)
+		(fields_autoplaced yes)
+		(stroke
+			(width 0.0006)
+			(type solid)
+		)
+		(fill
+			(color 0 0 0 0)
+		)
+		(property "Sheetname" "DAC"
+			(at 20.574 105.41 0)
+			(show_name no)
+			(do_not_autoplace no)
+			(effects
+				(font
+					(size 1.27 1.27)
+				)
+				(justify left bottom)
+			)
+		)
+		(property "Sheetfile" "dac.kicad_sch"
+			(at 20.574 133.35 0)
+			(show_name no)
+			(do_not_autoplace no)
+			(effects
+				(font
+					(size 1.27 1.27)
+				)
+				(justify left top)
+			)
+		)
+		(instances
+			(project "opentone"
+				(path "/0122bb8c-dbef-4db1-a6c6-9be780a38d9f"
+					(page "9")
+				)
+			)
+		)
 	)
 	(sheet

Commit message: started placing the components
Other:
- added sheet Touch (touch.kicad_sch)
Changed lines of the file:
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@@
+	)
+	(sheet
+		(at 160.02 22.86)
+		(size 50.8 25.4)
+		(exclude_from_sim no)
+		(in_bom yes)
+		(on_board yes)
+		(dnp no)
+		(fields_autoplaced yes)
+		(stroke
+			(width 0.1524)
+			(type solid)
+		)
+		(fill
+			(color 0 0 0 0)
+		)
+		(property "Sheetname" "Touch"
+			(at 160.02 22.1484 0)
+			(show_name no)
+			(do_not_autoplace no)
+			(effects
+				(font
+					(size 1.27 1.27)
+				)
+				(justify left bottom)
+			)
+		)
+		(property "Sheetfile" "touch.kicad_sch"
+			(at 160.02 48.8446 0)
+			(show_name no)
+			(do_not_autoplace no)
+			(effects
+				(font
+					(size 1.27 1.27)
+				)
+				(justify left top)
+			)
+		)
+		(instances
+			(project "opentone"
+				(path "/0122bb8c-dbef-4db1-a6c6-9be780a38d9f"
+					(page "10")
+				)
+			)
+		)
 	)
 	(sheet
