File: hardware/opentone/power.kicad_sch (KiCad schematic)
At the start: 60 parts, among them J3 LiPo JST-PH, Q1 AO3401A, Q2 AO3401A, U10 USBLC6-2SC6, U11 TPS63802DLAR, U12 MAX17048G+T10, U13 TPS7A2033PDBVR, U14 TPS7A2018PDBVR

Commit message: updated BOM
Parts:
- C64: value 22uF DNP -> 22uF; now not fitted
- C67: value 0.1uF -> 100nF
- R22: value 470 -> 470R
- R37: LCSC C227946 -> C23194; Manufacturer YAGEO -> UNI-ROYAL; Part number AC0603FR-07511KL -> 0603WAF5113T5E
- R38: LCSC C137671 -> C23265; Manufacturer YAGEO -> UNI-ROYAL; Part number RC0603FR-0791KL -> 0603WAF9102T5E
Changed lines of the file:
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@@
 		(on_board yes)
 		(in_pos_files yes)
-		(dnp no)
+		(dnp yes)
 		(property "Reference" "C64"
 			(at 182.626 149.098 0)
@@
 			)
 		)
-		(property "Value" "22uF DNP"
+		(property "Value" "22uF"
 			(at 187.198 153.67 0)
 			(show_name no)
@@
 			)
 		)
-		(property "Value" "0.1uF"
+		(property "Value" "100nF"
 			(at 218.694 149.606 0)
 			(show_name no)
@@
 			)
 		)
-		(property "Datasheet" "https://jlcpcb.com/api/file/downloadByFileSystemAccessId/8579706265439817728"
+		(property "Datasheet" "https://jlcpcb.com/api/file/downloadByFileSystemAccessId/8579706350726930432"
 			(at 41.91 68.58 0)
 			(hide yes)
@@
 			)
 		)
-		(property "Datasheet" "https://jlcpcb.com/api/file/downloadByFileSystemAccessId/8754855564801118208"
+		(property "Datasheet" "https://jlcpcb.com/api/file/downloadByFileSystemAccessId/8586178161256513537"
 			(at 168.91 139.7 0)
 			(hide yes)
@@
 			)
 		)
-		(property "Manufacturer" "YAGEO"
+		(property "Manufacturer" "UNI-ROYAL"
 			(at 168.91 139.7 0)
 			(hide yes)
@@
 			)
 		)
-		(property "Part number" "AC0603FR-07511KL"
+		(property "Part number" "0603WAF5113T5E"
 			(at 168.91 139.7 0)
 			(hide yes)
@@
 			)
 		)
-		(property "LCSC" "C227946"
+		(property "LCSC" "C23194"
 			(at 168.91 139.7 0)
 			(hide yes)
@@
 			)
 		)
-		(property "Datasheet" "https://jlcpcb.com/api/file/downloadByFileSystemAccessId/8755545249567514624"
+		(property "Datasheet" "https://jlcpcb.com/api/file/downloadByFileSystemAccessId/8579706328207712256"
 			(at 163.83 151.13 0)
 			(hide yes)
@@
 			)
 		)
-		(property "Manufacturer" "YAGEO"
+		(property "Manufacturer" "UNI-ROYAL"
 			(at 163.83 151.13 0)
 			(hide yes)
@@
 			)
 		)
-		(property "Part number" "RC0603FR-0791KL"
+		(property "Part number" "0603WAF9102T5E"
 			(at 163.83 151.13 0)
 			(hide yes)
@@
 			)
 		)
-		(property "LCSC" "C137671"
+		(property "LCSC" "C23265"
 			(at 163.83 151.13 0)
 			(hide yes)
@@
 			)
 		)
-		(property "Value" "470"
+		(property "Value" "470R"
 			(at 170.18 98.298 90)
 			(show_name no)

Commit message: started placing the components
Parts:
- added C70: 100nF, Capacitor_SMD:C_0603_1608Metric, symbol Device:C
- added R48: 470k, Resistor_SMD:R_0603_1608Metric, symbol Device:R
- F2: value ASMD1206-075 -> 1206L110THYR; LCSC C135339 -> C126818; Manufacturer Shenzhen JDT Fuse -> Littelfuse; Part number ASMD1206-075 -> 1206L110THYR
- R34: value 100k -> 47k; LCSC C25803 -> C25819; Part number 0603WAF1003T5E -> 0603WAF4702T5E
- R35: value 1M -> 100k; LCSC C22935 -> C25803; Part number 0603WAF1004T5E -> 0603WAF1003T5E
- R39: value 470k -> 1M; LCSC C23178 -> C22935; Part number 0603WAF4703T5E -> 0603WAF1004T5E
- USB1: value USB_C_Receptacle -> USB_C_Receptacle_USB2.0_16P; symbol Connector:USB_C_Receptacle -> Connector:USB_C_Receptacle_USB2.0_16P
Connections:
- net +3.3V: no longer R35.1
- net 3V3_EN: now also C70.1, R48.1
- net CHG_STAT: now also R35.1; no longer R35.2
- net GND: now also R35.2, C70.2, R48.2
- net USB_C_DM renamed USB_C_DN
- net USB_DM renamed USB_DN
- no-connect marks 11 -> 3
Other:
- moved on the sheet: R35
