File: hardware/opentone/screens.kicad_sch (KiCad schematic)
At the start: 41 parts, among them J201 LCD_ILI9341_TN_40P, J301 NHD-2.4-240320AF-CSXP, Q201 AO3400A, Q301 AO3400A, U201 MCP6001, U301 MCP6001

Commit message: added sd card, haptic, updated old parts and set a datasheet and MPN to all parts
Parts:
- C201, C301: footprint Capacitor_SMD:C_0805_2012Metric -> Capacitor_SMD:C_0603_1608Metric; LCSC (none) -> C19702; Manufacturer (none) -> Samsung Electro-Mechanics; Part number (none) -> CL10A106KP8NNNC
- C202, C204, C205, C302, C304, C305: footprint Capacitor_SMD:C_0805_2012Metric -> Capacitor_SMD:C_0603_1608Metric; LCSC (none) -> C14663; Manufacturer (none) -> YAGEO; Part number (none) -> CC0603KRX7R9BB104
- C203, C303: footprint Capacitor_SMD:C_0805_2012Metric -> Capacitor_SMD:C_0603_1608Metric; LCSC (none) -> C96446; Manufacturer (none) -> Samsung Electro-Mechanics; Part number (none) -> CL10A106MA8NRNC
- C206, C306: footprint Capacitor_SMD:C_0805_2012Metric -> Capacitor_SMD:C_0603_1608Metric; LCSC (none) -> C15849; Manufacturer (none) -> Samsung Electro-Mechanics; Part number (none) -> CL10A105KB8NNNC; now fitted
- FB201, FB301: footprint Inductor_SMD:L_0805_2012Metric -> Inductor_SMD:L_0603_1608Metric; LCSC (none) -> C1002; Manufacturer (none) -> Sunlord; Part number (none) -> GZ1608D601TF
- J201, J301: LCSC (none) -> C202114; Manufacturer (none) -> Hirose; Part number (none) -> FH12-40S-0.5SH(55)
- Q201, Q301: LCSC (none) -> C20917; Manufacturer (none) -> Alpha & Omega Semiconductor; Part number (none) -> AO3400A
- R201, R202, R203, R301, R302, R303, R304: footprint Resistor_SMD:R_0805_2012Metric -> Resistor_SMD:R_0603_1608Metric; LCSC (none) -> C23164; Manufacturer (none) -> UNI-ROYAL; Part number (none) -> 0603WAF470KT5E
- R211, R311: footprint Resistor_SMD:R_0805_2012Metric -> Resistor_SMD:R_0603_1608Metric; LCSC (none) -> C22775; Manufacturer (none) -> UNI-ROYAL; Part number (none) -> 0603WAF1000T5E
- R212, R312: footprint Resistor_SMD:R_0805_2012Metric -> Resistor_SMD:R_0603_1608Metric; LCSC (none) -> C22936; Manufacturer (none) -> UNI-ROYAL; Part number (none) -> 0603WAF100KT5E
- R213, R313: footprint Resistor_SMD:R_0805_2012Metric -> Resistor_SMD:R_0603_1608Metric; LCSC (none) -> C25803; Manufacturer (none) -> UNI-ROYAL; Part number (none) -> 0603WAF1003T5E
- R214: footprint Resistor_SMD:R_0805_2012Metric -> Resistor_SMD:R_0603_1608Metric; LCSC (none) -> C23206; Manufacturer (none) -> UNI-ROYAL; Part number (none) -> 0603WAF5602T5E
- R215, R315: footprint Resistor_SMD:R_0805_2012Metric -> Resistor_SMD:R_0603_1608Metric; LCSC (none) -> C21190; Manufacturer (none) -> UNI-ROYAL; Part number (none) -> 0603WAF1001T5E
- R314: footprint Resistor_SMD:R_0805_2012Metric -> Resistor_SMD:R_0603_1608Metric; LCSC (none) -> C23153; Manufacturer (none) -> UNI-ROYAL; Part number (none) -> 0603WAF3902T5E
- U201, U301: LCSC (none) -> C116490; Manufacturer (none) -> Microchip; Part number (none) -> MCP6001T-I/OT

Commit message: added recommendations from Teel s checklists
Parts:
- added C207, C307: 4n7, Capacitor_SMD:C_0603_1608Metric, symbol Device:C
- added R216, R316: 0R, Resistor_SMD:R_0603_1608Metric, symbol Device:R
Connections:
- net TFT1_BL_S: now also C207.2, R216.2; no longer Q201.2 (S), R212.1
- net TFT2_BL_S: now also C307.2, R316.2; no longer Q301.2 (S), R312.1
- net at R211.1, U201.1: now also C207.1
- net at R311.1, U301.1: now also C307.1
- new net: Q201.2 (S), R212.1, R216.1
- new net: Q301.2 (S), R312.1, R316.1

Commit message: license and datasheets script
Other:
- note added: "IPS panel: datasheets/display/NHD-2.4-240320AF-CSXP.pdf. LED 80-200 mA, Vf 2.7-3.4 V: at 82 mA from +3.3V the sink keeps ~0.2 V. Use VSYS if the current drops."
- note removed: "IPS panel: datasheets/NHD-2.4-240320AF-CSXP.pdf. LED 80-200 mA, Vf 2.7-3.4 V: at 82 mA from +3.3V the sink keeps ~0.2 V. Use VSYS if the current drops."
Changed lines of the file:
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@@
 		)
 	)
-	(text "IPS panel: datasheets/NHD-2.4-240320AF-CSXP.pdf. LED 80-200 mA, Vf 2.7-3.4 V: at 82 mA from +3.3V the sink keeps ~0.2 V. Use VSYS if the current drops."
+	(text "IPS panel: datasheets/display/NHD-2.4-240320AF-CSXP.pdf. LED 80-200 mA, Vf 2.7-3.4 V: at 82 mA from +3.3V the sink keeps ~0.2 V. Use VSYS if the current drops."
 		(exclude_from_sim no)
 		(at 208.28 203.2 0)

Commit message: updated BOM
Parts:
- C201, C203, C301, C303: value 10u -> 10uF
- C202, C204, C205, C302, C304, C305: value 100n -> 100nF
- C206, C306: value 1u -> 1uF
- C207, C307: value 4n7 -> 4.7nF
- R212, R312: value 1R 1% -> 1R
- R215, R315: value 1k 1% -> 1k
Changed lines of the file:
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@@
 			)
 		)
-		(property "Value" "10u"
+		(property "Value" "10uF"
 			(at 299.72 86.36 0)
 			(show_name no)
@@
 			)
 		)
-		(property "Value" "100n"
+		(property "Value" "100nF"
 			(at 317.5 116.84 0)
 			(show_name no)
@@
 			)
 		)
-		(property "Value" "100n"
+		(property "Value" "100nF"
 			(at 345.44 181.61 0)
 			(show_name no)
@@
 			)
 		)
-		(property "Value" "1u"
+		(property "Value" "1uF"
 			(at 280.67 186.69 0)
 			(show_name no)
@@
 			)
 		)
-		(property "Value" "1k 1%"
+		(property "Value" "1k"
 			(at 267.97 184.15 0)
 			(show_name no)
@@
 			)
 		)
-		(property "Value" "4n7"
+		(property "Value" "4.7nF"
 			(at 302.26 189.23 0)
 			(show_name no)
@@
 			)
 		)
-		(property "Value" "10u"
+		(property "Value" "10uF"
 			(at 119.38 116.84 0)
 			(show_name no)
@@
 			)
 		)
-		(property "Value" "10u"
+		(property "Value" "10uF"
 			(at 111.76 86.36 0)
 			(show_name no)
@@
 			)
 		)
-		(property "Value" "1u"
+		(property "Value" "1uF"
 			(at 92.71 186.69 0)
 			(show_name no)
@@
 			)
 		)
-		(property "Value" "10u"
+		(property "Value" "10uF"
 			(at 307.34 116.84 0)
 			(show_name no)
@@
 			)
 		)
-		(property "Value" "100n"
+		(property "Value" "100nF"
 			(at 309.88 86.36 0)
 			(show_name no)
@@
 			)
 		)
-		(property "Value" "4n7"
+		(property "Value" "4.7nF"
 			(at 114.3 189.23 0)
 			(show_name no)
@@
 			)
 		)
-		(property "Value" "1R 1%"
+		(property "Value" "1R"
 			(at 325.12 190.5 0)
 			(show_name no)
@@
 			)
 		)
-		(property "Value" "100n"
+		(property "Value" "100nF"
 			(at 157.48 181.61 0)
 			(show_name no)
@@
 			)
 		)
-		(property "Value" "1k 1%"
+		(property "Value" "1k"
 			(at 80.01 184.15 0)
 			(show_name no)
@@
 			)
 		)
-		(property "Value" "100n"
+		(property "Value" "100nF"
 			(at 121.92 86.36 0)
 			(show_name no)
@@
 			)
 		)
-		(property "Value" "1R 1%"
+		(property "Value" "1R"
 			(at 137.16 190.5 0)
 			(show_name no)
@@
 			)
 		)
-		(property "Value" "100n"
+		(property "Value" "100nF"
 			(at 129.54 116.84 0)
 			(show_name no)

Commit message: started placing the components
Parts:
- R217: renamed from FB201; value 600R/100MHz -> 0R; footprint Inductor_SMD:L_0603_1608Metric -> Resistor_SMD:R_0603_1608Metric; symbol Device:FerriteBead_Small -> Device:R_Small; LCSC C1002 -> C21189; Manufacturer Sunlord -> UNI-ROYAL; Part number GZ1608D601TF -> 0603WAF0000T5E
- R317: renamed from FB301; value 600R/100MHz -> 0R; footprint Inductor_SMD:L_0603_1608Metric -> Resistor_SMD:R_0603_1608Metric; symbol Device:FerriteBead_Small -> Device:R_Small; LCSC C1002 -> C21189; Manufacturer Sunlord -> UNI-ROYAL; Part number GZ1608D601TF -> 0603WAF0000T5E
Changed lines of the file:
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@@
 	)
 	(symbol
-		(lib_id "Device:FerriteBead_Small")
+		(lib_id "Device:R_Small")
 		(at 104.14 111.76 90)
 		(unit 1)
@@
 		(in_pos_files yes)
 		(dnp no)
-		(property "Reference" "FB201"
+		(property "Reference" "R217"
 			(at 101.6 109.22 90)
 			(show_name no)
@@
 			)
 		)
-		(property "Value" "600R/100MHz"
+		(property "Value" "0R"
 			(at 101.6 115.57 90)
 			(show_name no)
@@
 			)
 		)
-		(property "Footprint" "Inductor_SMD:L_0603_1608Metric"
+		(property "Footprint" "Resistor_SMD:R_0603_1608Metric"
 			(at 104.14 111.76 0)
 			(hide yes)
@@
 			)
 		)
-		(property "Datasheet" "https://jlcpcb.com/api/file/downloadByFileSystemAccessId/8579709915071365120"
+		(property "Datasheet" "https://jlcpcb.com/api/file/downloadByFileSystemAccessId/8756450222375747584"
 			(at 104.14 111.76 0)
 			(hide yes)
@@
 			)
 		)
-		(property "Description" ""
+		(property "Description" "Backlight LED supply: 0R (was a ferrite bead, the LED current is DC). Cut point for the backlight"
 			(at 104.14 111.76 0)
-			(show_name no)
-			(do_not_autoplace no)
-			(effects
-				(font
-					(size 1.27 1.27)
-				)
-			)
-		)
-		(property "Manufacturer" "Sunlord"
+			(hide yes)
+			(show_name no)
+			(do_not_autoplace no)
+			(effects
+				(font
+					(size 1.27 1.27)
+				)
+			)
+		)
+		(property "Manufacturer" "UNI-ROYAL"
 			(at 104.14 111.76 0)
 			(hide yes)
@@
 			)
 		)
-		(property "Part number" "GZ1608D601TF"
+		(property "Part number" "0603WAF0000T5E"
 			(at 104.14 111.76 0)
 			(hide yes)
@@
 			)
 		)
-		(property "LCSC" "C1002"
+		(property "LCSC" "C21189"
 			(at 104.14 111.76 0)
 			(hide yes)
@@
 			(project "opentone"
 				(path "/0122bb8c-dbef-4db1-a6c6-9be780a38d9f/89f9057f-f2b8-4b1e-8a19-f61bc42bac09"
-					(reference "FB201")
+					(reference "R217")
 					(unit 1)
 				)
@@
 	)
 	(symbol
-		(lib_id "Device:FerriteBead_Small")
+		(lib_id "Device:R_Small")
 		(at 292.1 111.76 90)
 		(unit 1)
@@
 		(in_pos_files yes)
 		(dnp no)
-		(property "Reference" "FB301"
+		(property "Reference" "R317"
 			(at 289.56 109.22 90)
 			(show_name no)
@@
 			)
 		)
-		(property "Value" "600R/100MHz"
+		(property "Value" "0R"
 			(at 289.56 115.57 90)
 			(show_name no)
@@
 			)
 		)
-		(property "Footprint" "Inductor_SMD:L_0603_1608Metric"
+		(property "Footprint" "Resistor_SMD:R_0603_1608Metric"
 			(at 292.1 111.76 0)
 			(hide yes)
@@
 			)
 		)
-		(property "Datasheet" "https://jlcpcb.com/api/file/downloadByFileSystemAccessId/8579709915071365120"
+		(property "Datasheet" "https://jlcpcb.com/api/file/downloadByFileSystemAccessId/8756450222375747584"
 			(at 292.1 111.76 0)
 			(hide yes)
@@
 			)
 		)
-		(property "Description" ""
+		(property "Description" "Backlight LED supply: 0R (was a ferrite bead, the LED current is DC). Cut point for the backlight"
 			(at 292.1 111.76 0)
-			(show_name no)
-			(do_not_autoplace no)
-			(effects
-				(font
-					(size 1.27 1.27)
-				)
-			)
-		)
-		(property "Manufacturer" "Sunlord"
+			(hide yes)
+			(show_name no)
+			(do_not_autoplace no)
+			(effects
+				(font
+					(size 1.27 1.27)
+				)
+			)
+		)
+		(property "Manufacturer" "UNI-ROYAL"
 			(at 292.1 111.76 0)
 			(hide yes)
@@
 			)
 		)
-		(property "Part number" "GZ1608D601TF"
+		(property "Part number" "0603WAF0000T5E"
 			(at 292.1 111.76 0)
 			(hide yes)
@@
 			)
 		)
-		(property "LCSC" "C1002"
+		(property "LCSC" "C21189"
 			(at 292.1 111.76 0)
 			(hide yes)
@@
 			(project "opentone"
 				(path "/0122bb8c-dbef-4db1-a6c6-9be780a38d9f/89f9057f-f2b8-4b1e-8a19-f61bc42bac09"
-					(reference "FB301")
-					(unit 1)
-				)
+					(reference "R317")
+					(unit 1)
+				)
