File: hardware/opentone/opentone.kicad_pcb (KiCad board)
At the start: 2 copper layers, 65 x 95.3 mm, 231 parts, among them J201 LCD_ILI9341_TN_40P, J3 LiPo JST-PH, J301 NHD-2.4-240320AF-CSXP, J401 SWD 2x5 1.27mm, J402 ST-LINK (Nucleo CN4), J403 Log UART4, J404 Spare GPIO, J501 Wheel FPC 0.5mm, J502 Wheel header, J601 DM3AT-SF-PEJM5, Q1 AO3401A, Q101 BSS138, Q201 AO3400A, Q301 AO3400A, SW401 RESET, SW402 BOOT0 (DFU), SW501 SKQGAFE010 Center, SW502 SKQGAFE010 Top, SW503 SKQGAFE010 Right, SW504 SKQGAFE010 Bottom, SW505 SKQGAFE010 Left, SW506 OFF / HOLD / ON, U10 USBLC6-2SC6, U101 FSC-BT1035, U102 TPS22917, U11 TPS63802DLAR, U12 MAX17048G+T10, U201 MCP6001, U301 MCP6001, U401 STM32F446VETx, U501 MPR121QR2, U601 APS6404L-3SQN-SN, U602 TPS22917, Y1 12.288MHz, Y401 8MHz, Y402 32.768kHz

Commit message: started placing the components
Parts:
- removed AP7312: AP7312-1833W6-7, Package_TO_SOT_SMD:SOT-23-6
- removed FB2: 600R@100MHz, Inductor_SMD:L_0603_1608Metric
- removed FB201, FB301: 600R/100MHz, Inductor_SMD:L_0603_1608Metric
- added C1201: 4.7uF, Capacitor_SMD:C_0603_1608Metric, B.Cu at (98.3, 152.5)
- added C1202: 100pF, Capacitor_SMD:C_0603_1608Metric, B.Cu at (96.8, 152.5)
- added C1203: 2.2uF, Capacitor_SMD:C_0603_1608Metric, B.Cu at (92.3, 152.5)
- added C1204: 100pF, Capacitor_SMD:C_0603_1608Metric, B.Cu at (90.8, 152.5)
- added C1205: 2.2uF, Capacitor_SMD:C_0603_1608Metric, B.Cu at (95.3, 152.5)
- added C1206: 100pF, Capacitor_SMD:C_0603_1608Metric, B.Cu at (93.8, 152.5)
- added C207: 4.7nF, Capacitor_SMD:C_0603_1608Metric, F.Cu at (162.5, 96.8)
- added C307: 4.7nF, Capacitor_SMD:C_0603_1608Metric, F.Cu at (160.5, 132.0)
- added C504: 1uF, Capacitor_SMD:C_0603_1608Metric, F.Cu at (110.5, 101.5)
- added C505: 100nF, Capacitor_SMD:C_0603_1608Metric, F.Cu at (115.5, 101.3)
- added C506: 1uF, Capacitor_SMD:C_0603_1608Metric, F.Cu at (111.5, 110.0)
- added C68: 1uF, Capacitor_SMD:C_0603_1608Metric, F.Cu at (99.8, 160.0)
- added C69: 1uF, Capacitor_SMD:C_0603_1608Metric, F.Cu at (106.0, 160.5)
- added C70: 100nF, Capacitor_SMD:C_0603_1608Metric, F.Cu at (118.7, 141.5)
- added C701: 1uF, Capacitor_SMD:C_0603_1608Metric, B.Cu at (52.5, 114.5)
- added C702: 1uF, Capacitor_SMD:C_0603_1608Metric, B.Cu at (36.1, 113.1)
- added C703: 4.7uF, Capacitor_SMD:C_0603_1608Metric, B.Cu at (52.8, 117.5)
- added C704: 100nF, Capacitor_SMD:C_0603_1608Metric, B.Cu at (52.8, 116.0)
- added C705: 100nF, Capacitor_SMD:C_0603_1608Metric, B.Cu at (57.0, 111.5)
- added C706: 100nF, Capacitor_SMD:C_0603_1608Metric, B.Cu at (66.0, 116.0)
- added C707: 2.2uF, Capacitor_SMD:C_0603_1608Metric, B.Cu at (66.0, 118.0)
- added C708: 2.2uF, Capacitor_SMD:C_0603_1608Metric, B.Cu at (58.5, 111.5)
- added C709: 22uF, Capacitor_SMD:C_0805_2012Metric, B.Cu at (66.5, 113.5)
- added C710: 22uF, Capacitor_SMD:C_0805_2012Metric, B.Cu at (67.0, 121.5)
- added C711: 2.2uF, Capacitor_SMD:C_0603_1608Metric, B.Cu at (67.0, 123.5)
- added C712: 2.2uF, Capacitor_SMD:C_0603_1608Metric, B.Cu at (63.5, 121.5)
- added C713: 2.2uF, Capacitor_SMD:C_0603_1608Metric, B.Cu at (52.8, 120.5)
- added C714: 2.2uF, Capacitor_SMD:C_0603_1608Metric, B.Cu at (58.5, 122.5)
- added C715: 2.2uF, Capacitor_SMD:C_0603_1608Metric, B.Cu at (55.0, 118.0)
- added C716: 2.2uF, Capacitor_SMD:C_0603_1608Metric, B.Cu at (56.0, 121.5)
- added C717: 100nF, Capacitor_SMD:C_0603_1608Metric, B.Cu at (57.1, 95.5)
- added C718: 100nF, Capacitor_SMD:C_0603_1608Metric, B.Cu at (52.8, 119.0)
- added C719: 100nF, Capacitor_SMD:C_0603_1608Metric, B.Cu at (72.2, 106.9)
- added D401: STATUS, LED_SMD:LED_0603_1608Metric, F.Cu at (-41.8, 108.0)
- added D701: TPD1E10B06DPYR, Package_SON:Texas_DPY0002A_0.6x1mm_P0.65mm, B.Cu at (50.0, 95.2)
- added D702: TPD1E10B06DPYR, Package_SON:Texas_DPY0002A_0.6x1mm_P0.65mm, B.Cu at (35.5, 85.6)
- added D703: TPD1E10B06DPYR, Package_SON:Texas_DPY0002A_0.6x1mm_P0.65mm, B.Cu at (42.5, 99.6)
- added D8: SMF5.0A, Diode_SMD:D_SOD-123F, F.Cu at (151.0, 156.8)
- added JP1201: IQS drain, Jumper:SolderJumper-2_P1.3mm_Bridged_RoundedPad1.0x1.5mm, B.Cu at (102.8, 153.5)
- added JP1202: Wheel top, Jumper:SolderJumper-3_P1.3mm_Bridged12_RoundedPad1.0x1.5mm, B.Cu at (85.3, 152.0)
- added JP1203: Wheel right, Jumper:SolderJumper-3_P1.3mm_Bridged12_RoundedPad1.0x1.5mm, B.Cu at (85.3, 149.5)
- added JP1204: Wheel bottom, Jumper:SolderJumper-3_P1.3mm_Bridged12_RoundedPad1.0x1.5mm, B.Cu at (85.3, 147.0)
- added JP1205: Wheel left, Jumper:SolderJumper-3_P1.3mm_Bridged12_RoundedPad1.0x1.5mm, B.Cu at (85.3, 144.5)
- added JP1206: Wheel center, Jumper:SolderJumper-3_P1.3mm_Bridged12_RoundedPad1.0x1.5mm, B.Cu at (85.3, 142.0)
- added JP502: Haptic drain, Jumper:SolderJumper-2_P1.3mm_Bridged_RoundedPad1.0x1.5mm, F.Cu at (106.0, 102.3)
- added JP6: VS1053 drain, Jumper:SolderJumper-2_P1.3mm_Bridged_RoundedPad1.0x1.5mm, F.Cu at (96.2, 161.0)
- added JP701: DAC drain, Jumper:SolderJumper-2_P1.3mm_Bridged_RoundedPad1.0x1.5mm, B.Cu at (44.5, 114.6)
- added Jack2: SJ-43515TS-SMT-TR, opentone:CUI_SJ-43515TS-SMT-TR, B.Cu at (47.1, 80.0)
- added NT1: GND-GNDA, NetTie:NetTie-2_SMD_Pad0.5mm, F.Cu at (109.8, 159.5)
- added NT701: HP2 ground, NetTie:NetTie-2_SMD_Pad0.5mm, B.Cu at (52.0, 83.1)
- added Q2: AO3401A, Package_TO_SOT_SMD:SOT-23, F.Cu at (118.2, 171.8)
- added R1201: 470R, Resistor_SMD:R_0603_1608Metric, B.Cu at (90.3, 149.5)
- added R1202: 470R, Resistor_SMD:R_0603_1608Metric, B.Cu at (90.0, 148.0)
- added R1203: 470R, Resistor_SMD:R_0603_1608Metric, B.Cu at (90.3, 146.5)
- added R1204: 470R, Resistor_SMD:R_0603_1608Metric, B.Cu at (90.3, 145.0)
- added R1205: 470R, Resistor_SMD:R_0603_1608Metric, B.Cu at (90.3, 143.5)
- added R1206: 4.7k, Resistor_SMD:R_0603_1608Metric, B.Cu at (100.3, 147.5)
- added R216: 0R, Resistor_SMD:R_0603_1608Metric, F.Cu at (164.0, 96.6)
- added R217: 0R, Resistor_SMD:R_0603_1608Metric, F.Cu at (169.8, 92.2)
- added R316: 0R, Resistor_SMD:R_0603_1608Metric, F.Cu at (162.5, 137.0)
- added R317: 0R, Resistor_SMD:R_0603_1608Metric, F.Cu at (171.2, 121.6)
- added R4: 47k, Resistor_SMD:R_0603_1608Metric, B.Cu at (85.1, 100.1)
- added R404: 1k, Resistor_SMD:R_0603_1608Metric, F.Cu at (-38.5, 108.0)
- added R48: 470k, Resistor_SMD:R_0603_1608Metric, F.Cu at (118.7, 140.0)
- added R509: 100k, Resistor_SMD:R_0603_1608Metric, F.Cu at (114.5, 110.0)
- added R701: 100k, Resistor_SMD:R_0603_1608Metric, B.Cu at (42.4, 118.6)
- added R702: 200k, Resistor_SMD:R_0603_1608Metric, B.Cu at (63.7, 106.4)
- added R703: 4.7k, Resistor_SMD:R_0603_1608Metric, B.Cu at (71.7, 109.4)
- added R704: 4.7k, Resistor_SMD:R_0603_1608Metric, B.Cu at (71.7, 110.9)
- added R705: 100k, Resistor_SMD:R_0603_1608Metric, B.Cu at (52.5, 111.5)
- added R706: 10k, Resistor_SMD:R_0603_1608Metric, B.Cu at (52.5, 110.0)
- added R8: 100k, Resistor_SMD:R_0603_1608Metric, F.Cu at (98.8, 153.0)
- added TP1201: IQS_MCLR, TestPoint:TestPoint_Pad_D1.0mm, B.Cu at (103.8, 149.0)
- added TP2: VSYS, TestPoint:TestPoint_Pad_D1.0mm, F.Cu at (131.8, 139.0)
- added TP3: VBAT, TestPoint:TestPoint_Pad_D1.0mm, F.Cu at (127.1, 166.8)
- added TP4: +3.3V, TestPoint:TestPoint_Pad_D1.0mm, F.Cu at (116.3, 153.0)
- added TP5: +1V8, TestPoint:TestPoint_Pad_D1.0mm, F.Cu at (105.3, 157.5)
- added TP501: M+, TestPoint:TestPoint_Pad_1.5x1.5mm, F.Cu at (110.5, 95.3)
- added TP502: M-, TestPoint:TestPoint_Pad_1.5x1.5mm, F.Cu at (114.5, 95.3)
- added TP6: +3.3VA, TestPoint:TestPoint_Pad_D1.0mm, F.Cu at (109.8, 147.0)
- added U1201: IQS7222A, Package_DFN_QFN:VQFN-20-1EP_3x3mm_P0.4mm_EP1.7x1.7mm, B.Cu at (94.8, 147.8)
- added U13: TPS7A2033PDBVR, Package_TO_SOT_SMD:SOT-23-5, F.Cu at (102.7, 152.1)
- added U14: TPS7A2018PDBVR, Package_TO_SOT_SMD:SOT-23-5, F.Cu at (102.5, 163.0)
- added U15: TPD4E05U06DQAR, Package_SON:USON-10_2.5x1.0mm_P0.5mm, B.Cu at (90.6, 104.7)
- added U502: DRV2605L, Package_SO:VSSOP-10_3x3mm_P0.5mm, F.Cu at (113.0, 105.0)
- added U701: CS43131-CNZ, Package_DFN_QFN:TQFN-40-1EP_5x5mm_P0.4mm_EP3.5x3.5mm, B.Cu at (60.0, 117.0)
- added U702: TPS7A2018PDBVR, Package_TO_SOT_SMD:SOT-23-5, B.Cu at (39.7, 115.6)
- added U703: SN74AVC4T245PWR, Package_SO:TSSOP-16_4.4x5mm_P0.65mm, B.Cu at (58.9, 101.6)
- added U704: PCA9306DCUR, Package_SO:VSSOP-8_2.3x2mm_P0.5mm, B.Cu at (67.1, 108.6)
- C101, C201, C203, C301, C303, C605: value 10u -> 10uF
- C102, C103, C202, C204, C205, C302, C304, C305, C401, C402, C403, C404, C405, C406, C408, C410, C417, C601, C606: value 100n -> 100nF
- C104, C105, C107, C113, C206, C306, C409, C603: value 1u -> 1uF
- C108, C604: value 1n -> 1nF
- C29, C3, C30, C31, C32, C33, C34, C35, C36, C37, C38, C39, C40, C41, C42, C43, C44, C45, C9, JP501, Jack1, R16, R17, R18, R41, R42, R43, R44, R45, R46, R47, R501, R503, R504, R505, R506, R507, SW501, SW502, SW503, SW504, VS1, Y1: moved to B.Cu
- C407, C602: value 4.7u -> 4.7uF
- C411, C412: value 2.2u -> 2.2uF
- C413, C414: value 15p -> 15pF
- C415, C416: value 6.8p -> 6.8pF
- C501, C503: value 100n -> 100nF; moved to B.Cu
- C502: value 1u -> 1uF; moved to B.Cu
- C64: value 22uF DNP -> 22uF
- C67: value 0.1uF -> 100nF
- F2: value ASMD1206-075 -> 1206L110THYR
- J201, J301: moved to F.Cu
- L3: value 0.47uH XFL4015-471ME -> 0.47uH DFE252012P-R47M; footprint Inductor_SMD:L_Coilcraft_XAL4020-XXX -> Inductor_SMD:L_1008_2520Metric_Pad1.43x2.20mm_HandSolder
- R13: value 10 -> 10R; moved to B.Cu
- R14, R2: value 20 -> 20R; moved to B.Cu
- R212, R312: value 1R 1% -> 1R
- R215, R315: value 1k 1% -> 1k
- R22: value 470 -> 470R
- R3: value 100K -> 100k; moved to B.Cu
- R34: value 10k -> 47k
- R39: value 470k -> 1M
- R502: value 75k 1% -> 75k; moved to B.Cu
- R6: value 47k -> 100k
- R7: value 47k -> 100k; moved to B.Cu
- USB1: value USB_C_Receptacle -> USB_C_Receptacle_USB2.0_16P
- moved R617 224.4 mm to (70.5, 157.6), turned to -90 degrees
- moved R616 221.9 mm to (75.0, 157.5), turned to -90 degrees
- moved R620 221.7 mm to (69.0, 157.6), turned to -90 degrees
- moved R615 220.9 mm to (78.0, 157.6), turned to -90 degrees
- moved R32 219.1 mm to (162.5, 169.8)
- moved R610 218.9 mm to (71.8, 153.0), turned to 180 degrees
- moved R612 217.2 mm to (73.5, 157.6), turned to -90 degrees
- moved R614 215.7 mm to (72.0, 157.6), turned to -90 degrees
- moved R618 214.2 mm to (81.0, 157.6), turned to -90 degrees
- moved R20 214.2 mm to (157.7, 167.5), turned to 90 degrees
- moved R619 214.1 mm to (79.5, 157.6), turned to -90 degrees
- moved R613 213.3 mm to (76.5, 157.6), turned to -90 degrees
- moved R19 212.5 mm to (153.5, 167.8), turned to 90 degrees
- moved SW503 211.9 mm to (40.1, 156.7), turned to 180 degrees
- moved R30 210.6 mm to (156.5, 157.7), turned to 90 degrees
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Connections:
- net /MCU/SPARE_PA2 renamed IQS_RDY
- net /MCU/SPARE_PC13 renamed /MCU/STATUS_LED
- net /Memory/PSRAM_VDD renamed Net-(JP601-B)
- net /Memory/SD_3V3_IN renamed Net-(JP602-B)
- net Net-(JP2-A) renamed /Power/3V3_REG
- net Net-(JP3-A) renamed /Power/PROG_2K
- net Net-(JP3-B) renamed /Power/PROG_10K
- net Net-(JP3-C) renamed /Power/PROG
- net Net-(U11-FB) renamed /Power/3V3_FB
- net Net-(VS1-GBUF) renamed /Audio/HP_GBUF
- net Net-(VS1-LEFT) renamed /Audio/HP_L
- net Net-(VS1-RIGHT) renamed /Audio/HP_R
- C40 pad 1: +3.3V -> +3.3VA
- C42 pad 1: +3.3V -> +3.3VA
- C44 pad 1: +3.3V -> +3.3VA
- C45 pad 1: +3.3V -> +3.3VA
- C52 pad 1: +1V8 -> /Power/AVDD_LDO
- C65 pad 1: VSYS -> /Power/VS_VIN
- J501 pad 1: /Buttons/WHEEL_TOP -> WHEEL_TOP
- J501 pad 2: /Buttons/WHEEL_RIGHT -> WHEEL_RIGHT
- J501 pad 3: /Buttons/WHEEL_BOTTOM -> WHEEL_BOTTOM
- J501 pad 4: /Buttons/WHEEL_LEFT -> WHEEL_LEFT
- J501 pad 6: /Buttons/WHEEL_CENTER -> WHEEL_CENTER
- J502 pad 1: /Buttons/WHEEL_TOP -> WHEEL_TOP
- J502 pad 2: /Buttons/WHEEL_RIGHT -> WHEEL_RIGHT
- J502 pad 3: /Buttons/WHEEL_BOTTOM -> WHEEL_BOTTOM
- J502 pad 4: /Buttons/WHEEL_LEFT -> WHEEL_LEFT
- J502 pad 6: /Buttons/WHEEL_CENTER -> WHEEL_CENTER
- JP1 pad 1: Net-(J3-Pin_1) -> Net-(JP1-A)
- Q201 pad 2: /Screens/TFT1_BL_S -> Net-(Q201-S)
- Q301 pad 2: /Screens/TFT2_BL_S -> Net-(Q301-S)
- R212 pad 1: /Screens/TFT1_BL_S -> Net-(Q201-S)
- R3 pad 1: +3.3V -> +3.3VA
- R312 pad 1: /Screens/TFT2_BL_S -> Net-(Q301-S)
- R35 pad 1: +3.3V -> CHG_STAT
- R35 pad 2: CHG_STAT -> GND
- R6 pad 1: VBUS -> Net-(Q2-G)
- R6 pad 2: VBUS_SENSE -> GND
- U10 pad 6: /Power/USB_C_DP -> unconnected-(U10-I/O1-Pad6)
- U401 pad 69: HP2_DET -> DAC_INT
- U501 pad 10: /Buttons/WHEEL_TOP -> MPR_WHEEL_TOP
- U501 pad 11: /Buttons/WHEEL_BOTTOM -> MPR_WHEEL_BOTTOM
- U501 pad 12: /Buttons/WHEEL_CENTER -> MPR_WHEEL_CENTER
- U501 pad 8: /Buttons/WHEEL_RIGHT -> MPR_WHEEL_RIGHT
- U501 pad 9: /Buttons/WHEEL_LEFT -> MPR_WHEEL_LEFT
- VS1 pad 14: +3.3V -> +3.3VA
- VS1 pad 19: +3.3V -> +3.3VA
- VS1 pad 27: VTX -> unconnected-(VS1-TX-Pad27)
- VS1 pad 32: +3.3V -> +3.3VA
- VS1 pad 6: +3.3V -> +3.3VA
- bat-man1 pad 9: (no net) -> GND
Routing:
- removed copper zone on B.Cu, net GND
Other:
- board size 65 x 95.3 mm -> 150 x 100.5 mm
- copper layers 2 -> 4

Commit message: wire the main MCU caps
Parts:
- C60, R32: moved to B.Cu
- moved R3 55.3 mm to (93.8, 66.7)
- moved R44 55.3 mm to (93.8, 68.2)
- moved C30 54.2 mm to (90.0, 64.0)
- moved C37 54.2 mm to (90.0, 61.0)
- moved C43 54.2 mm to (90.0, 65.5)
- moved C44 54.2 mm to (90.0, 62.5)
- moved R43 54.2 mm to (89.8, 59.5)
- moved R16 54.1 mm to (85.2, 63.0)
- moved R17 54.1 mm to (85.2, 61.5)
- moved C31 54.0 mm to (100.2, 72.2)
- moved C32 54.0 mm to (109.5, 64.0)
- moved C33 54.0 mm to (97.5, 57.5)
- moved C35 54.0 mm to (97.2, 72.0)
- moved C39 54.0 mm to (109.5, 62.5)
- moved C40 54.0 mm to (109.5, 65.5)
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Connections:
- net /Power/USB_C_DM renamed /Power/USB_C_DN
- net USB_DM renamed USB_DN
- U10 pad 6: unconnected-(U10-I/O1-Pad6) -> /Power/USB_C_DP
Routing:
- net USB_DP: track 0.00 -> 65.8 mm
- net USB_DN: track 0.00 -> 65.2 mm
- net /Power/VBUS_IN: track 0.00 -> 47.6 mm
- net GND: track 0.00 -> 42.2 mm, vias 0 -> 33
- net /MCU/MCU_3V3: track 0.00 -> 21.0 mm
- net /Power/USB_C_DP: track 0.00 -> 16.1 mm
- net /Power/USB_C_DN: track 0.00 -> 14.5 mm
- net Net-(USB1-SHIELD): track 0.00 -> 14.4 mm
- net VBAT: track 0.00 -> 14.3 mm
- net /Power/3V3_REG: track 0.00 -> 11.4 mm
- net /MCU/MCU_VDDA: track 0.00 -> 10.3 mm
- net /MCU/HSE_OUT: track 0.00 -> 10.0 mm
- net 3V3_EN: track 0.00 -> 9.04 mm
- net /MCU/HSE_IN: track 0.00 -> 7.87 mm
- net /MCU/LSE_IN: track 0.00 -> 7.00 mm
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- added copper zone on In1.Cu, net GND

Commit message: wired screens and vs1053
Parts:
- R7: moved to F.Cu
- moved J502 81.1 mm to (37.0, 149.0), turned to 180 degrees
- moved C40 59.2 mm to (78.5, 116.0), turned to -90 degrees
- moved C37 58.1 mm to (70.0, 115.5), turned to -90 degrees
- moved NT1 55.8 mm to (68.1, 122.5)
- moved C69 53.9 mm to (66.4, 124.0)
- moved JP6 53.9 mm to (56.6, 124.5)
- moved TP5 53.9 mm to (65.7, 121.0)
- moved U14 53.9 mm to (62.9, 126.5)
- moved C68 53.9 mm to (60.2, 123.5)
- moved C33 52.6 mm to (70.5, 102.7), turned to 90 degrees
- moved R45 52.0 mm to (83.5, 113.5)
- moved R3 51.4 mm to (67.0, 110.5), turned to 0 degrees
- moved R44 51.4 mm to (67.0, 112.0)
- moved C32 50.7 mm to (83.5, 107.5)
- moved C39 50.7 mm to (83.5, 106.0)
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Routing:
- net GND: track 42.2 -> 216.5 mm, vias 33 -> 137
- net TFT_DC: track 0.00 -> 157.4 mm, vias 0 -> 2
- net TFT_D0: track 0.00 -> 136.0 mm, vias 0 -> 4
- net TFT_D2: track 0.00 -> 135.5 mm, vias 0 -> 4
- net TFT_D1: track 0.00 -> 135.4 mm, vias 0 -> 4
- net TFT_WR: track 0.00 -> 134.6 mm, vias 0 -> 4
- net TFT_D6: track 0.00 -> 128.7 mm, vias 0 -> 6
- net TFT_D4: track 0.00 -> 127.0 mm, vias 0 -> 4
- net TFT_D5: track 0.00 -> 126.4 mm, vias 0 -> 4
- net TFT_D11: track 0.00 -> 120.5 mm, vias 0 -> 4
- net TFT_D10: track 0.00 -> 119.6 mm, vias 0 -> 4
- net TFT_D7: track 0.00 -> 119.5 mm, vias 0 -> 5
- net TFT_D9: track 0.00 -> 118.2 mm, vias 0 -> 4
- net TFT_D8: track 0.00 -> 118.1 mm, vias 0 -> 4
- net TFT_D13: track 0.00 -> 117.6 mm, vias 0 -> 4
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- added copper zone on In2.Cu, net +3.3V
- added copper zone on In2.Cu, net +3.3VA
- added copper zone on In1.Cu, net GNDA
- added copper zone on In2.Cu, net VSYS

Commit message: update clickwheel footprint and wired the board more
Parts:
- moved JP6 89.8 mm to (-30.5, 102.5)
- moved TP6 66.0 mm to (60.2, 110.5)
- moved C66 62.7 mm to (64.5, 117.0)
- moved FB3 62.5 mm to (61.7, 116.2)
- moved JP4 61.6 mm to (60.2, 113.0)
- moved C52 60.8 mm to (56.7, 113.0)
- moved U13 60.0 mm to (54.5, 116.3)
- moved C65 59.4 mm to (51.5, 113.7)
- moved R45 44.1 mm to (118.3, 86.5), turned to 180 degrees
- moved R46 43.5 mm to (118.3, 89.0), turned to 180 degrees
- moved R505 35.5 mm to (44.3, 152.5)
- moved R506 29.0 mm to (52.5, 167.0)
- moved C711 27.7 mm to (37.8, 106.0), turned to 180 degrees
- moved U703 24.3 mm to (18.3, 109.6)
- moved C710 24.2 mm to (37.8, 108.0), turned to 0 degrees
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Routing:
- net GNDA: track 27.6 -> 178.4 mm
- net BTN_RIGHT: track 0.00 -> 120.5 mm, vias 0 -> 1
- net BTN_TOP: track 0.00 -> 112.1 mm, vias 0 -> 1
- net BTN_CENTER: track 0.00 -> 103.9 mm, vias 0 -> 1
- net LOCK_SW: track 0.00 -> 101.0 mm, vias 0 -> 2
- net SD_CD: track 6.26 -> 103.4 mm
- net BTN_BOTTOM: track 0.00 -> 95.9 mm, vias 0 -> 1
- net BTN_LEFT: track 0.00 -> 91.3 mm, vias 0 -> 1
- net TFT_D3: track 51.9 -> 133.2 mm, vias 3 -> 4
- net 3V3_EN: track 11.5 -> 89.7 mm
- net HP1_DET: track 17.2 -> 84.2 mm, vias 2 -> 5
- net GND: track 216.5 -> 275.8 mm, vias 137 -> 171
- net CHG_STAT: track 1.35 -> 57.8 mm, vias 0 -> 2
- net VSYS: track 90.9 -> 147.2 mm, vias 6 -> 7
- net I2S_SCLK: track 4.95 -> 58.8 mm, vias 0 -> 1
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- added copper zone on F.Cu, net /Power/3V3_REG
- added copper zone on F.Cu, net VSYS
- removed copper zone on In1.Cu, net GNDA
